File: led_clock.kicad_pcb (KiCad board)
At the start: 2 copper layers, 121.3 x 139.7 mm, 328 parts, among them J1 Programming (ICSP), J2 USB_B_Micro, J3 Barrel_Jack, Q1 2N7002, SW1 SW_Push, SW2 SW_Push, SW3 SW_Push, SW4 SW_SPDT, U1 MPM3620A, U2 TLV70032_SOT23-5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

Commit message: Center PCB
Parts:
- moved C100 176.5 mm to (150.0, 122.7)
- moved C11 176.5 mm to (142.8, 97.5)
- moved C110 176.5 mm to (193.3, 129.3)
- moved C112 176.5 mm to (189.0, 118.9)
- moved C12 176.5 mm to (147.3, 91.7)
- moved C128 176.5 mm to (189.0, 97.0)
- moved C129 176.5 mm to (189.5, 92.9)
- moved C130 176.5 mm to (193.3, 86.6)
- moved C131 176.5 mm to (196.7, 79.9)
- moved C133 176.5 mm to (177.6, 72.4)
- moved C140 176.5 mm to (153.7, 87.5)
- moved C141 176.5 mm to (150.0, 93.2)
- moved C19 176.5 mm to (151.6, 57.4)
- moved C22 176.5 mm to (131.4, 50.9)
- moved C30 176.5 mm to (129.0, 85.6)
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Other:
- board text added: "LED Clock"
